Commit message: Buggs Solved
Removed Hand's random vibration+Tuned PID power grip+ImprovedContactFlickering+TaxelsTrans Correction

File: Gazebo_Simulation/World/Allegro_Hand/allegro_hand_description_right.urdf (robot description, URDF)
Before this commit: robot allegro_hand_right, 38 links, 37 joints
Links:
- link boh_bracket: geometry collision mesh filename=package://allegro_hand_description/meshes/part_4.dae; visual mesh filename=package://allegro_hand_description/meshes/part_4.dae
- link palm_bracket: geometry collision mesh filename=package://allegro_hand_description/meshes/palm_bracket.dae; visual mesh filename=package://allegro_hand_description/meshes/palm_bracket.dae
Joints:
- joint joint_0_0: limit effort=1 velocity=20 -> lower=-1.57 upper=1.57 effort=15 velocity=20
- joint joint_10_0: limit effort=1 velocity=20 -> lower=0 upper=1.57 effort=15 velocity=20
- joint joint_11_0: limit effort=1 velocity=20 -> lower=0 upper=1.57 effort=15 velocity=20
- joint joint_12_0: limit effort=1 velocity=20 -> lower=0 upper=1.57 effort=15 velocity=20
- joint joint_13_0: limit effort=1 velocity=20 -> lower=0 upper=2 effort=15 velocity=20
- joint joint_14_0: limit effort=1 velocity=20 -> lower=0 upper=1.57 effort=15 velocity=20
- joint joint_15_0: limit effort=1 velocity=20 -> lower=0 upper=1.57 effort=15 velocity=20
- joint joint_1_0: limit effort=1 velocity=20 -> lower=0 upper=1.57 effort=15 velocity=20
- joint joint_2_0: limit effort=1 velocity=20 -> lower=0 upper=1.57 effort=15 velocity=20
- joint joint_3_0: limit effort=1 velocity=20 -> lower=0 upper=1.57 effort=15 velocity=20
- joint joint_4_0: limit effort=1 velocity=20 -> lower=-1.57 upper=1.57 effort=15 velocity=20
- joint joint_5_0: limit effort=1 velocity=20 -> lower=0 upper=1.57 effort=15 velocity=20
- joint joint_6_0: limit effort=1 velocity=20 -> lower=0 upper=1.57 effort=15 velocity=20
- joint joint_7_0: limit effort=1 velocity=20 -> lower=0 upper=1.57 effort=15 velocity=20
- joint joint_8_0: limit effort=1 velocity=20 -> lower=-1.57 upper=1.57 effort=15 velocity=20
- joint joint_9_0: limit effort=1 velocity=20 -> lower=0 upper=1.57 effort=15 velocity=20

Commit message: Added the fingertip sensors
Added the fingetip sensors taxels coordinates to the data structure

File: Gazebo_Simulation/World/Allegro_Hand/allegro_hand_description_right.urdf (robot description, URDF)
Before this commit: robot allegro_hand_right, 38 links, 37 joints
Links:
- link imf_bracket: geometry collision mesh filename=package://allegro_hand_description/meshes/medial_front.dae; visual mesh filename=package://allegro_hand_description/meshes/medial_front.dae
- link ipf_bracket: geometry collision mesh filename=package://allegro_hand_description/meshes/proximal_front.dae; visual mesh filename=package://allegro_hand_description/meshes/proximal_front.dae
- link mmf_bracket: geometry collision mesh filename=package://allegro_hand_description/meshes/medial_front.dae; visual mesh filename=package://allegro_hand_description/meshes/medial_front.dae
- link mpf_bracket: geometry collision mesh filename=package://allegro_hand_description/meshes/proximal_front.dae; visual mesh filename=package://allegro_hand_description/meshes/proximal_front.dae
- link pmf_bracket: geometry collision mesh filename=package://allegro_hand_description/meshes/medial_front.dae; visual mesh filename=package://allegro_hand_description/meshes/medial_front.dae
- link ppf_bracket: geometry collision mesh filename=package://allegro_hand_description/meshes/proximal_front.dae; visual mesh filename=package://allegro_hand_description/meshes/proximal_front.dae

Commit message: Initial Taxels Activation Detection Algo + RVIZ Debugging

File: Gazebo_Simulation/World/Allegro_Hand/allegro_hand_description_right.urdf (robot description, URDF)
Before this commit: robot allegro_hand_right, 38 links, 37 joints
Links:
- added link boh, mass 0.00784811; collision mesh filename=package://allegro_hand_description/meshes/boh_fpcb.stl; visual mesh filename=package://allegro_hand_description/meshes/boh_fpcb.stl
- added link index_fingertip_main_fpcb, mass 0.00142203; collision mesh filename=package://allegro_hand_description/meshes/distal_fpcb_1.stl; visual mesh filename=package://allegro_hand_description/meshes/distal_fpcb_1.stl
- added link index_fingertip_side_fpcb, mass 0.00128609; collision mesh filename=package://allegro_hand_description/meshes/distal_fpcb_2.stl; visual mesh filename=package://allegro_hand_description/meshes/distal_fpcb_2.stl
- added link index_medial_back_fpcb, mass 0.000991462; collision mesh filename=package://allegro_hand_description/meshes/medial_back_fpcb.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; visual mesh filename=package://allegro_hand_description/meshes/medial_back_fpcb.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
- added link index_medial_front_fpcb, mass 0.00086951; collision mesh filename=package://allegro_hand_description/meshes/medial_front_fpcb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; visual mesh filename=package://allegro_hand_description/meshes/medial_front_fpcb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
- added link index_proximal_back_fpcb, mass 0.00110296; collision mesh filename=package://allegro_hand_description/meshes/proximal_back_fpc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; visual mesh filename=package://allegro_hand_description/meshes/proximal_back_fpc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
- added link index_proximal_front_fpcb, mass 0.000871809; collision mesh filename=package://allegro_hand_description/meshes/proximal_frontfpc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; visual mesh filename=package://allegro_hand_description/meshes/proximal_frontfpc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
- added link middle_fingertip_main_fpcb, mass 0.00142203; collision mesh filename=package://allegro_hand_description/meshes/distal_fpcb_1.stl; visual mesh filename=package://allegro_hand_description/meshes/distal_fpcb_1.stl
- added link middle_fingertip_side_fpcb, mass 0.00128609; collision mesh filename=package://allegro_hand_description/meshes/distal_fpcb_2.stl; visual mesh filename=package://allegro_hand_description/meshes/distal_fpcb_2.stl
- added link middle_medial_back_fpcb, mass 0.000991462; collision mesh filename=package://allegro_hand_description/meshes/medial_back_fpcb.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; visual mesh filename=package://allegro_hand_description/meshes/medial_back_fpcb.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
- added link middle_medial_front_fpcb, mass 0.00086951; collision mesh filename=package://allegro_hand_description/meshes/medial_front_fpcb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; visual mesh filename=package://allegro_hand_description/meshes/medial_front_fpcb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
- added link middle_proximal_back_fpcb, mass 0.00110296; collision mesh filename=package://allegro_hand_description/meshes/proximal_back_fpc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; visual mesh filename=package://allegro_hand_description/meshes/proximal_back_fpc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
- added link middle_proximal_front_fpcb, mass 0.000871809; collision mesh filename=package://allegro_hand_description/meshes/proximal_frontfpc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; visual mesh filename=package://allegro_hand_description/meshes/proximal_frontfpc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
- added link palm_fpcb, mass 0.00098458; collision mesh filename=package://allegro_hand_description/meshes/palm_fpcb.stl; visual mesh filename=package://allegro_hand_description/meshes/palm_fpcb.stl
- added link pinky_fingertip_main_fpcb, mass 0.00142203; collision mesh filename=package://allegro_hand_description/meshes/distal_fpcb_1.stl; visual mesh filename=package://allegro_hand_description/meshes/distal_fpcb_1.stl
- added link pinky_fingertip_side_fpcb, mass 0.00128609; collision mesh filename=package://allegro_hand_description/meshes/distal_fpcb_2.stl; visual mesh filename=package://allegro_hand_description/meshes/distal_fpcb_2.stl
- added link pinky_medial_back_fpcb, mass 0.000991462; collision mesh filename=package://allegro_hand_description/meshes/medial_back_fpcb.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; visual mesh filename=package://allegro_hand_description/meshes/medial_back_fpcb.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
- added link pinky_medial_front_fpcb, mass 0.00086951; collision mesh filename=package://allegro_hand_description/meshes/medial_front_fpcb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; visual mesh filename=package://allegro_hand_description/meshes/medial_front_fpcb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
- added link pinky_proximal_back_fpcb, mass 0.00110296; collision mesh filename=package://allegro_hand_description/meshes/proximal_back_fpc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; visual mesh filename=package://allegro_hand_description/meshes/proximal_back_fpc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
- added link pinky_proximal_front_fpcb, mass 0.000871809; collision mesh filename=package://allegro_hand_description/meshes/proximal_frontfpc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; visual mesh filename=package://allegro_hand_description/meshes/proximal_frontfpc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
- added link thumb_fingertip_main_fpcb, mass 0.00142203; collision mesh filename=package://allegro_hand_description/meshes/distal_fpcb_1.stl; visual mesh filename=package://allegro_hand_description/meshes/distal_fpcb_1.stl
- added link thumb_fingertip_side_fpcb, mass 0.00128609; collision mesh filename=package://allegro_hand_description/meshes/distal_fpcb_2.stl; visual mesh filename=package://allegro_hand_description/meshes/distal_fpcb_2.stl
- added link thumb_medial_back_fpcb, mass 0.000612423; collision mesh filename=package://allegro_hand_description/meshes/part_5.stl; visual mesh filename=package://allegro_hand_description/meshes/part_5.stl
- added link thumb_medial_front_fpcb, mass 0.000462123; collision mesh filename=package://allegro_hand_description/meshes/part_6.stl; visual mesh filename=package://allegro_hand_description/meshes/part_6.stl
- link boh_bracket: geometry collision mesh filename=package://allegro_hand_description/meshes/part_4.stl; visual mesh filename=package://allegro_hand_description/meshes/part_4.stl
- link imf_bracket: geometry collision mesh filename=package://allegro_hand_description/meshes/medial_front.stl; visual mesh filename=package://allegro_hand_description/meshes/medial_front.stl
- link ipf_bracket: geometry collision mesh filename=package://allegro_hand_description/meshes/proximal_front.stl; visual mesh filename=package://allegro_hand_description/meshes/proximal_front.stl
- link mmf_bracket: geometry collision mesh filename=package://allegro_hand_description/meshes/medial_front.stl; visual mesh filename=package://allegro_hand_description/meshes/medial_front.stl
- link mpf_bracket: geometry collision mesh filename=package://allegro_hand_description/meshes/proximal_front.stl; visual mesh filename=package://allegro_hand_description/meshes/proximal_front.stl
- link palm_bracket: geometry collision mesh filename=package://allegro_hand_description/meshes/palm_bracket.stl; visual mesh filename=package://allegro_hand_description/meshes/palm_bracket.stl
- link pmf_bracket: geometry collision mesh filename=package://allegro_hand_description/meshes/medial_front.stl; visual mesh filename=package://allegro_hand_description/meshes/medial_front.stl
- link ppf_bracket: geometry collision mesh filename=package://allegro_hand_description/meshes/proximal_front.stl; visual mesh filename=package://allegro_hand_description/meshes/proximal_front.stl
Joints:
- added joint joint_boh: type fixed, parent boh_bracket, child boh, origin xyz=0.019996 -0.0318962 -0.0093 rpy=0 -0 0, axis 0 0 1, limit effort=1 velocity=20
- added joint joint_index_fingertip_main_fpcb: type fixed, parent ift_bracket, child index_fingertip_main_fpcb, origin xyz=0.00776046 -0.01766 0.0135 rpy=3.95134e-15 -6.07352e-15 -3.889e-30, axis 0 0 1, limit effort=1 velocity=20
- added joint joint_index_fingertip_side_fpcb: type fixed, parent ift_bracket, child index_fingertip_side_fpcb, origin xyz=0.0399163 0.0096 -0.00275858 rpy=-3.14159 1.29682e-17 1.10568e-30, axis 0 0 1, limit effort=1 velocity=20
- added joint joint_index_medial_back_fpcb: type fixed, parent imb_bracket, child index_medial_back_fpcb, origin xyz=0.0337 0.0105 -1.73472e-16 rpy=-1.5708 4.62281e-16 -1.5708, axis 0 0 1, limit effort=1 velocity=20
- added joint joint_index_medial_front_fpcb: type fixed, parent imf_bracket, child index_medial_front_fpcb, origin xyz=0.0337 0.0089 0.0044 rpy=1.5708 -4.84955e-31 1.5708, axis 0 0 1, limit effort=1 velocity=20
- added joint joint_index_proximal_back_fpcb: type fixed, parent ipb_bracket, child index_proximal_back_fpcb, origin xyz=-0.0277 0.0099 0.0009 rpy=-1.5708 -1.40936e-17 -4.33377e-16, axis 0 0 1, limit effort=1 velocity=20
- added joint joint_index_proximal_front_fpcb: type fixed, parent ipf_bracket, child index_proximal_front_fpcb, origin xyz=0.0319 0.00595201 0.0044 rpy=1.69568e-14 4.09448e-18 3.98238e-32, axis 0 0 1, limit effort=1 velocity=20
- added joint joint_middle_fingertip_main_fpcb: type fixed, parent mft_bracket, child middle_fingertip_main_fpcb, origin xyz=0.00776046 -0.01766 0.0135 rpy=-4.82947e-15 -7.14706e-15 2.77556e-17, axis 0 0 1, limit effort=1 velocity=20
- added joint joint_middle_fingertip_side_fpcb: type fixed, parent mft_bracket, child middle_fingertip_side_fpcb, origin xyz=0.0399163 0.0096 -0.00275858 rpy=3.14159 -1.38778e-17 -2.77556e-17, axis 0 0 1, limit effort=1 velocity=20
- added joint joint_middle_medial_back_fpcb: type fixed, parent mmb_bracket, child middle_medial_back_fpcb, origin xyz=0.0337 0.0105 1.38778e-17 rpy=-1.5708 2.57582e-26 -1.5708, axis 0 0 1, limit effort=1 velocity=20
- added joint joint_middle_medial_front_fpcb: type fixed, parent mmf_bracket, child middle_medial_front_fpcb, origin xyz=0.0337 0.0089 0.0044 rpy=1.5708 1.79259e-30 1.5708, axis 0 0 1, limit effort=1 velocity=20
- added joint joint_middle_proximal_back_fpcb: type fixed, parent mpb_bracket, child middle_proximal_back_fpcb, origin xyz=-0.0277 0.0099 0.0009 rpy=-1.5708 1.69768e-31 -2.34367e-30, axis 0 0 1, limit effort=1 velocity=20
- added joint joint_middle_proximal_front_fpcb: type fixed, parent mpf_bracket, child middle_proximal_front_fpcb, origin xyz=0.0319 0.00595201 0.0044 rpy=-6.26539e-15 -5.20417e-18 5.55112e-17, axis 0 0 1, limit effort=1 velocity=20
- added joint joint_palm_fpcb: type fixed, parent palm_bracket, child palm_fpcb, origin xyz=-0.0202546 -0.088 -0.006 rpy=0 -0 0, axis 0 0 1, limit effort=1 velocity=20
- added joint joint_pinky_fingertip_main_fpcb: type fixed, parent pft_bracket, child pinky_fingertip_main_fpcb, origin xyz=0.00776046 -0.01766 0.0135 rpy=-4.08652e-17 5.17584e-16 1.66533e-16, axis 0 0 1, limit effort=1 velocity=20
- added joint joint_pinky_fingertip_side_fpcb: type fixed, parent pft_bracket, child pinky_fingertip_side_fpcb, origin xyz=0.0399163 0.0096 -0.00275858 rpy=-3.14159 5.15965e-17 5.55112e-17, axis 0 0 1, limit effort=1 velocity=20
- added joint joint_pinky_medial_back_fpcb: type fixed, parent pmb_bracket, child pinky_medial_back_fpcb, origin xyz=0.0337 0.0105 -4.51028e-17 rpy=-1.5708 4.44891e-19 -1.5708, axis 0 0 1, limit effort=1 velocity=20
- added joint joint_pinky_medial_front_fpcb: type fixed, parent pmf_bracket, child pinky_medial_front_fpcb, origin xyz=0.0337 0.0089 0.0044 rpy=1.5708 -4.44891e-19 1.5708, axis 0 0 1, limit effort=1 velocity=20
- added joint joint_pinky_proximal_back_fpcb: type fixed, parent ppb_bracket, child pinky_proximal_back_fpcb, origin xyz=-0.0277 0.0099 0.0009 rpy=-1.5708 -8.3852e-18 -7.27119e-30, axis 0 0 1, limit effort=1 velocity=20
- added joint joint_pinky_proximal_front_fpcb: type fixed, parent ppf_bracket, child pinky_proximal_front_fpcb, origin xyz=0.0319 0.00595201 0.0044 rpy=-5.00673e-15 6.88757e-19 -5.55112e-17, axis 0 0 1, limit effort=1 velocity=20
- added joint joint_thumb_fingertip_main_fpcb: type fixed, parent tft_bracket, child thumb_fingertip_main_fpcb, origin xyz=0.00776046 -0.01766 0.0135 rpy=8.63584e-16 -5.01319e-16 5.12794e-18, axis 0 0 1, limit effort=1 velocity=20
- added joint joint_thumb_fingertip_side_fpcb: type fixed, parent tft_bracket, child thumb_fingertip_side_fpcb, origin xyz=0.0399163 0.0096 -0.00275858 rpy=-3.14159 -9.5307e-16 5.18075e-18, axis 0 0 1, limit effort=1 velocity=20
- added joint joint_thumb_medial_back_fpcb: type fixed, parent tmb_bracket, child thumb_medial_back_fpcb, origin xyz=-0.0108 0.0277 -2.68882e-17 rpy=-1.5708 7.27098e-31 -7.93211e-15, axis 0 0 1, limit effort=1 velocity=20
- added joint joint_thumb_medial_front_fpcb: type fixed, parent tmf_bracket, child thumb_medial_front_fpcb, origin xyz=0.0100023 -0.0277 0.007 rpy=-1.5708 -5.1393e-32 5.59764e-15, axis 0 0 1, limit effort=1 velocity=20
- joint joint_10_0: origin xyz=-0.054 1.8735e-16 6.93889e-18 rpy=1.89044e-16 -3.19266e-15 -2.31621e-15 -> xyz=-0.054 1.38778e-17 -1.249e-16 rpy=7.38677e-17 -5.80172e-16 -7.55426e-16
- joint joint_11_0: limit lower=0 upper=1.57 effort=15 velocity=20 -> lower=0 upper=2.5 effort=15 velocity=20; origin xyz=-0.04615 6.93889e-18 0.0001 rpy=9.68157e-16 1.44316e-15 -1.10006e-18 -> xyz=-0.04615 2.08167e-17 0.0001 rpy=-2.08897e-16 7.34965e-16 -9.23803e-14
- joint joint_14_0: origin xyz=0.0119 0 0.02545 rpy=-3.14159 1.5708 0 -> xyz=0.0119 -1.38778e-17 0.02545 rpy=3.14159 1.5708 0
- joint joint_15_0: origin xyz=-0.0514 -9.89486e-15 -0.0001 rpy=7.8724e-16 1.94208e-15 2.09209e-13 -> xyz=-0.0514 -9.00668e-15 -0.0001 rpy=-4.53557e-16 3.39461e-16 2.07948e-13
- joint joint_1_0: limit lower=0 upper=1.57 effort=15 velocity=20 -> lower=0 upper=2.5 effort=15 velocity=20; origin xyz=0 -0.0119 0.02545 rpy=-1.5708 -1.5708 0 -> xyz=6.93889e-18 -0.0119 0.02545 rpy=-1.5708 -1.5708 0
- joint joint_2_0: origin xyz=0.054 -2.08167e-17 0 rpy=3.51153e-16 -1.76861e-16 -3.14159 -> xyz=0.054 2.28983e-16 7.63278e-17 rpy=-1.93545e-14 4.22599e-15 -3.14159
- joint joint_3_0: limit lower=0 upper=1.57 effort=15 velocity=20 -> lower=0 upper=2.5 effort=15 velocity=20; origin xyz=-0.04615 1.38778e-17 0.0001 rpy=2.47521e-16 -2.87243e-16 -9.91762e-14 -> xyz=-0.04615 2.77556e-17 0.0001 rpy=-4.33522e-16 1.57792e-15 -7.74196e-17
- joint joint_5_0: limit lower=0 upper=1.57 effort=15 velocity=20 -> lower=0 upper=2.5 effort=15 velocity=20; origin xyz=6.93889e-18 -0.0119 0.02545 rpy=-1.5708 1.5708 0 -> xyz=-4.16334e-17 -0.0119 0.02545 rpy=-1.5708 1.5708 0
- joint joint_6_0: origin xyz=-0.054 2.56739e-16 -1.76074e-15 rpy=5.58159e-16 -7.32724e-16 -3.32379e-15 -> xyz=-0.054 -1.66533e-16 -7.30319e-16 rpy=2.4529e-15 -5.42863e-15 3.19463e-15
- joint joint_7_0: limit lower=0 upper=1.57 effort=15 velocity=20 -> lower=0 upper=2.5 effort=15 velocity=20; origin xyz=-0.04615 2.08167e-17 0.0001 rpy=7.63278e-16 5.80199e-16 -9.4334e-27 -> xyz=-0.04615 2.77556e-17 0.0001 rpy=-6.02043e-15 5.70882e-15 9.18658e-14
- joint joint_9_0: limit lower=0 upper=1.57 effort=15 velocity=20 -> lower=0 upper=2.5 effort=15 velocity=20; origin xyz=-2.77556e-17 -0.0119 0.02545 rpy=-1.5708 1.5708 0 -> xyz=-1.38778e-17 -0.0119 0.02545 rpy=-1.5708 1.5708 0
- joint joint_index_fingertip_bracket: origin xyz=-0.0135 0.004 0.0254 rpy=-3.14159 -1.01255e-15 -3.14159 -> xyz=-0.0135 0.004 0.0254 rpy=3.14159 -5.14611e-15 3.14159
- joint joint_index_medial_back_bracket: origin xyz=-0.0215 0.004 0.0259 rpy=-3.14159 -1.66749e-15 3.14159 -> xyz=-0.0215 0.004 0.0259 rpy=3.14159 4.76628e-16 -3.14159
- joint joint_index_medial_front_bracket: origin xyz=-0.0215 -0.004 -0.0021 rpy=1.55523e-28 1.64355e-17 -3.14159 -> xyz=-0.0215 -0.004 -0.0021 rpy=6.04764e-19 8.37023e-19 3.14159
- joint joint_index_proximal_back_bracket: origin xyz=0.0249 -0.0037 0.0253 rpy=-3.14159 1.75587e-16 3.12083e-29 -> xyz=0.0249 -0.0037 0.0253 rpy=-3.14159 -4.95527e-15 -2.49458e-28
- joint joint_index_proximal_front_bracket: origin xyz=0.0249 0.0077 -0.0017 rpy=-5.29761e-14 6.49973e-18 -2.65051e-30 -> xyz=0.0249 0.0077 -0.0017 rpy=1.74055e-15 -7.22547e-16 -8.65583e-16
- joint joint_middle_fingertip_bracket: origin xyz=-0.0135 0.004 0.0254 rpy=-3.14159 -5.9952e-15 -3.14159 -> xyz=-0.0135 0.004 0.0254 rpy=3.14159 -8.32667e-16 -3.14159
- joint joint_middle_medial_back_bracket: origin xyz=-0.0215 0.004 0.0259 rpy=-3.14159 -9.53737e-16 3.14159 -> xyz=-0.0215 0.004 0.0259 rpy=-3.14159 -1.5933e-17 3.14159
- joint joint_middle_medial_front_bracket: origin xyz=-0.0215 -0.004 -0.0021 rpy=-4.39991e-17 5.71587e-18 3.14159 -> xyz=-0.0215 -0.004 -0.0021 rpy=-2.91434e-16 2.19124e-17 3.14159
- joint joint_middle_proximal_back_bracket: origin xyz=-0.0249 0.0037 0.0253 rpy=3.14159 -5.25942e-17 -3.14159 -> xyz=-0.0249 0.0037 0.0253 rpy=-3.14159 4.05868e-15 3.14159
- joint joint_middle_proximal_front_bracket: origin xyz=-0.0249 -0.0077 -0.0017 rpy=-5.38894e-32 -1.09608e-17 3.14159 -> xyz=-0.0249 -0.0077 -0.0017 rpy=-1.96804e-15 3.74674e-16 3.14159
- joint joint_pinky_fingertip_bracket: origin xyz=-0.0135 0.004 0.0254 rpy=-3.14159 -6.33477e-16 -3.14159 -> xyz=-0.0135 0.004 0.0254 rpy=3.14159 4.4328e-16 3.14159
- joint joint_pinky_medial_back_bracket: origin xyz=-0.0215 0.004 0.0259 rpy=3.14159 -4.42051e-16 3.14159 -> xyz=-0.0215 0.004 0.0259 rpy=-3.14159 -1.31932e-17 3.14159
- joint joint_pinky_medial_front_bracket: origin xyz=-0.0215 -0.004 -0.0021 rpy=-4.41528e-16 3.94696e-17 3.14159 -> xyz=-0.0215 -0.004 -0.0021 rpy=5.55513e-32 -1.31932e-17 3.14159
- joint joint_pinky_proximal_back_bracket: origin xyz=-0.0249 0.0037 0.0253 rpy=3.14159 2.21409e-15 3.14159 -> xyz=-0.0249 0.0037 0.0253 rpy=-3.14159 5.61195e-15 3.14159
- joint joint_pinky_proximal_front_bracket: origin xyz=-0.0249 -0.0077 -0.0017 rpy=-1.19862e-14 1.01475e-15 3.14159 -> xyz=-0.0249 -0.0077 -0.0017 rpy=-1.96935e-15 3.88558e-16 3.14159
- joint joint_thumb_fingertip_bracket: origin xyz=-0.0291 0.0037 0.0253 rpy=3.14159 3.0723e-15 -3.14159 -> xyz=-0.0291 0.0037 0.0253 rpy=3.14159 5.80134e-16 -3.14159
- joint joint_thumb_medial_back_bracket: origin xyz=-0.0249 0.004 -0.0022 rpy=-2.32122e-16 2.56368e-16 -1.5708 -> xyz=-0.0249 0.004 -0.0022 rpy=-6.46681e-16 -1.5186e-15 -1.5708
- joint joint_thumb_medial_front_bracket: origin xyz=-0.0249 -0.004 0.0258 rpy=3.14159 -1.54748e-16 -1.5708 -> xyz=-0.0249 -0.004 0.0258 rpy=3.14159 -7.73741e-17 -1.5708
