Commit message: Integration of Allegro with UR5e

File: ROS_WS/robot_arm_ws/src/coro_workstations/coro_descriptions/urdf/common/2f_coupling.urdf.xacro (robot description, xacro)
@@ -2,44 +2,41 @@
 <robot name="2f_coupling" xmlns:xacro="http://ros.org/wiki/xacro">
 	<xacro:macro name="coupling_robotiq_2f" params="parent prefix *origin">
+	<link name="ur_bracket">
+		<visual>
+			<origin xyz="0 0 0" rpy="0 -0 0" />
+			<geometry>
+			<mesh filename="package://coro_descriptions/meshes/ur_bracket.stl"/>
+			</geometry>
+			<material name="ur_bracket_material">
+			<color rgba="0.615686 0.811765 0.929412 1.0"/>
+			</material>
+		</visual>
+		<collision>
+			<origin xyz="0 0 0" rpy="0 -0 0" />
+			<geometry>
+			<mesh filename="package://coro_descriptions/meshes/ur_bracket.stl"/>
+			</geometry>
+			<material name="ur_bracket_material">
+			<color rgba="0.615686 0.811765 0.929412 1.0"/>
+			</material>
+		</collision>
+		<inertial>
+			<origin xyz="0.0271498 0.0180673 -0.00967187" rpy="0 0 0"/>
+			<mass value="0.05307" />
+			<inertia ixx="1.71151e-05" ixy="0"  ixz="0" iyy="1.50513e-05" iyz="1.25799e-06" izz="2.94394e-05" />
+		</inertial>
+	</link>
 		<!-- Mount the coupling to the robot side -->
-	        <joint name="${prefix}coupling_robot_fix" type="fixed">
+	    <joint name="${prefix}coupling_robot_fix" type="fixed">
 			<xacro:insert_block name="origin" />
-	            	<parent link="${parent}" />
-            		<child link="${prefix}2f_coupling" />
-	        </joint>
-	        <!-- Coupling -->
-		<link name="${prefix}2f_coupling">
-			<visual>
-				<origin xyz="0 0 0" rpy="0 0 0" />
-				<geometry>
-	                    		<cylinder length="0.017" radius="0.0375"/>
-	                	</geometry>
-	                	<material name="Robotiq-Black">
-	                    		<color rgba="0.2 0.2 0.2 1.0"/>
-	                	</material>
-			</visual>
-	            	<collision>
-	                	<origin xyz="0 0 0" rpy="0 0 0" />
-	                	<geometry>
-	                    		<cylinder length="0.017" radius="0.0375"/>
-	                	</geometry>
-	            	</collision>
-	            	<inertial>
-	                	<origin xyz="0 0 0" rpy="0 0 0"/>
-	                	<mass value="0.150"/>
-	                	<inertia ixx="0.000056" ixy="0"        ixz="0"
-	                	         iyx="0"        iyy="0.000056" iyz="0"
-	                	         izx="0"        izy="0"        izz="0.000105"/>
-	            	</inertial>
-	        </link>
-	        <gazebo reference="${prefix}2f_coupling">
-    			<material>Gazebo/Black</material>
-  		</gazebo>
-	        <!-- Mount the gripper to the coupling -->
-	        <link name="${prefix}coupling_gripper_fix"/>
-	        <joint name="coupling_to_gripper" type="fixed">
-	        	<parent link="${prefix}2f_coupling"/>
-	        	<child link="${prefix}coupling_gripper_fix"/>
-	        	<origin xyz="0 0 -0.0054" rpy="0 0 0"/>
+	            <parent link="${parent}" />
+            	<child link="${prefix}ur_bracket" />
+	    </joint>
+	    <!-- Mount the gripper to the coupling -->
+	    <link name="${prefix}coupling_gripper_fix"/>
+	    <joint name="coupling_to_gripper" type="fixed">
+	        <parent link="${prefix}ur_bracket"/>
+	        <child link="${prefix}coupling_gripper_fix"/>
+	        <origin xyz="0 0 0" rpy="0 0 0"/>
 		</joint>
 	</xacro:macro>

File: ROS_WS/robot_arm_ws/src/coro_workstations/coro_descriptions/urdf/workstations/ur5e_workstation.urdf.xacro (robot description, xacro)
@@ -23,11 +23,11 @@
 	<xacro:include filename="$(find coro_descriptions)/urdf/common/2f_coupling.urdf.xacro"/>
 	<xacro:coupling_robotiq_2f prefix="" parent="tool0">
-		<origin xyz="0 0 0.0045" rpy="0 0 1.5708"/>
+		<origin xyz="0 0 0.01" rpy="0 0 0"/>
 	</xacro:coupling_robotiq_2f>
 	<!-- GRIPPER -->
-	<xacro:include filename="$(find robotiq_85_description)/urdf/robotiq_85_gripper.urdf.xacro"/>
-	<xacro:robotiq_85_gripper prefix="" parent="coupling_gripper_fix">
-		<origin xyz="0 0 0.0108" rpy="0 -1.5708 0"/>
-	</xacro:robotiq_85_gripper>
+	<xacro:include filename="$(find allegro_hand_gazebo)/allegro_hand_description/urdf/allegro_hand_description_right.urdf.xacro"/>
+	<xacro:allegro_hand_right prefix="" parent="coupling_gripper_fix">
+		<origin xyz="0 -0.041 0.105" rpy="0 0 0"/>
+	</xacro:allegro_hand_right>
 	<link name="tcp"/>
 	<joint name="tcp_to_gripper" type="fixed">
@@ -36,4 +36,35 @@
 		<origin xyz="0 0 0.165" rpy="0 0 0"/>
 	</joint>
+	<!-- OBJECT TO GRASP -->
+    <link name="cubic_object_link">
+		<visual>
+		<origin xyz="0 0 0" rpy="0 -0 1.5708" />
+		<geometry>
+		<mesh filename="package://coro_descriptions/meshes/cubic_object.stl"/>
+		</geometry>
+		<material name="link_testing_cube_material">
+		<color rgba="0.615686 0.811765 0.929412 1.0"/>
+		</material>
+		</visual>
+		<collision>
+		<origin xyz="0 0 0" rpy="0 -0 1.5708" />
+		<geometry>
+		<mesh filename="package://coro_descriptions/meshes/cubic_object.stl"/>
+		</geometry>
+		<material name="link_testing_cube_material">
+		<color rgba="0.615686 0.811765 0.929412 1.0"/>
+		</material>
+		</collision>
+		<inertial>
+		<origin xyz="-1.02566e-17 9.23364e-19 0.1075" rpy="0 0 0"/>
+		<mass value="0.0770781" />
+		<inertia ixx="0.000307188" ixy="0"  ixz="0" iyy="0.000307188" iyz="0" izz="2.05542e-05" />
+		</inertial>
+    </link>
+	<joint name='object_to_table' type='fixed'>
+		<origin xyz="0.004217 -0.201201 0.951750" rpy="0 0 0"/>
+    	<parent link="table_base"/>
+    	<child link="cubic_object_link"/>
+    </joint>
 	<!-- GAZEBO -->
 	<gazebo>
