Commit message: Added code for synthetic data generation
I added a python script , service nodes for data saving and ur5e workstation reset in the simulation environment. Also, I have optimized the control to achieve a good grasp from only one angle of approach

File: ROS_WS/robot_arm_ws/src/coro_workstations/allegro_hand/allegro_hand_simulation/allegro_hand_gazebo/allegro_hand_description/urdf/allegro_hand_description_right.urdf.xacro (robot description, xacro)
@@ -236,5 +236,5 @@
                 <child link="link_3" />
                 <axis xyz="0 0 1"/>
-                <limit effort="15" velocity="20" lower="0" upper="1.4" />
+                <limit effort="15" velocity="20" lower="0" upper="1.47" />
                 <dynamics damping="1" friction="0.5" />
                 <gazebo>
@@ -787,5 +787,5 @@
                 <child link="link_7" />
                 <axis xyz="0 0 1"/>
-                <limit effort="15" velocity="20" lower="0" upper="1.4" />
+                <limit effort="15" velocity="20" lower="0" upper="1.47" />
                 <dynamics damping="1" friction="0.5" />
                 <gazebo>
@@ -1338,5 +1338,5 @@
                 <child link="link_11" />
                 <axis xyz="0 0 1"/>
-                <limit effort="15" velocity="20" lower="0" upper="1.4" />
+                <limit effort="15" velocity="20" lower="0" upper="1.47" />
                 <dynamics damping="1" friction="0.5" />
                 <gazebo>

File: ROS_WS/robot_arm_ws/src/coro_workstations/coro_descriptions/urdf/workstations/ur5e_workstation.urdf (robot description, URDF)
Before this commit: robot ur5e_2f85, 78 links, 77 joints
Links:
- added link cubic_object_link, mass 0.0770781; collision mesh filename=package://coro_descriptions/meshes/cubic_object.stl; visual mesh filename=package://coro_descriptions/meshes/cubic_object.stl
Joints:
- added joint object_to_table: type fixed, parent table_base, child cubic_object_link, origin xyz=0.004217 -0.201201 0.951750 rpy=0 0 0
- joint joint_0_0: limit lower=-1.57 upper=1.57 effort=15 velocity=20 -> lower=-0.45 upper=0.55 effort=15 velocity=20
- joint joint_10_0: limit lower=0 upper=1.57 effort=15 velocity=20 -> lower=0 upper=1.5 effort=15 velocity=20
- joint joint_11_0: limit lower=0 upper=2.5 effort=15 velocity=20 -> lower=0 upper=1.47 effort=15 velocity=20
- joint joint_12_0: limit lower=0 upper=1.57 effort=15 velocity=20 -> lower=0.35 upper=1.57 effort=15 velocity=20
- joint joint_13_0: limit lower=0 upper=2 effort=15 velocity=20 -> lower=-1.3 upper=1.15 effort=15 velocity=20
- joint joint_14_0: limit lower=0 upper=1.57 effort=15 velocity=20 -> lower=0 upper=1.45 effort=15 velocity=20
- joint joint_15_0: limit lower=0 upper=1.57 effort=15 velocity=20 -> lower=0 upper=1.7 effort=15 velocity=20
- joint joint_1_0: limit lower=0 upper=2.5 effort=15 velocity=20 -> lower=0 upper=1.65 effort=15 velocity=20
- joint joint_2_0: limit lower=0 upper=1.57 effort=15 velocity=20 -> lower=0 upper=1.5 effort=15 velocity=20
- joint joint_3_0: limit lower=0 upper=2.5 effort=15 velocity=20 -> lower=0 upper=1.47 effort=15 velocity=20
- joint joint_4_0: limit lower=-1.57 upper=1.57 effort=15 velocity=20 -> lower=-0.55 upper=0.45 effort=15 velocity=20
- joint joint_5_0: limit lower=0 upper=2.5 effort=15 velocity=20 -> lower=0 upper=1.65 effort=15 velocity=20
- joint joint_6_0: limit lower=0 upper=1.57 effort=15 velocity=20 -> lower=0 upper=1.5 effort=15 velocity=20
- joint joint_7_0: limit lower=0 upper=2.5 effort=15 velocity=20 -> lower=0 upper=1.47 effort=15 velocity=20
- joint joint_8_0: limit lower=-1.57 upper=1.57 effort=15 velocity=20 -> lower=-0.45 upper=0.55 effort=15 velocity=20
- joint joint_9_0: limit lower=0 upper=2.5 effort=15 velocity=20 -> lower=0 upper=1.65 effort=15 velocity=20
- joint wrist_3_joint: origin xyz=0 0.0996 -2.042830148012698e-11 rpy=1.570796326589793 3.141592653589793 3.141592653589793 -> xyz=0 0.0996 -2.042830148012698e-11 rpy=1.570796326589793 4.71238898018 3.141592653589793
