Commit message: Emergency Backup push

File: ROS_WS/robot_arm_ws/src/coro_workstations/coro_descriptions/urdf/workstations/ur5e_workstation.urdf (robot description, URDF)
Before this commit: robot ur5e_2f85, 79 links, 78 joints
Links:
- added link table_top, mass 1.88145; collision mesh filename=package://coro_descriptions/meshes/table_top.stl; visual mesh filename=package://coro_descriptions/meshes/table_top.stl
Joints:
- added joint table_top_to_table_base: type fixed, parent table_base, child table_top, origin xyz=0.004217 -0.201201 0.97025 rpy=0 0 1.57
- joint coupling_robot_fix: origin xyz=0 0 0.01 rpy=0 0 0 -> xyz=0 0 0.01 rpy=0 0 1.5707963267948966
- joint object_to_table: origin xyz=0.004217 -0.201201 0.951750 rpy=0 0 0 -> xyz=0.004217 -0.201201 1.016225 rpy=0 0 0

File: ROS_WS/robot_arm_ws/src/coro_workstations/coro_descriptions/urdf/workstations/ur5e_workstation.urdf.xacro (robot description, xacro)
@@ -11,4 +11,34 @@
 		<child link="table_base"/>
 		<origin xyz="0 0 0" rpy="0 0 0"/>
+	</joint>
+	<!-- Table top -->
+	<link name='table_top'>
+		<inertial>
+			<origin xyz="1.41182e-16 -6.13716e-17 -0.00229716" rpy="0 0 0"/>
+			<mass value="1.88145" />
+			<inertia ixx="0.132708" ixy="0"  ixz="0" iyy="0.0587177" iyz="0" izz="0.191419" />
+		</inertial>
+		<collision>
+			<origin xyz="0 0 -0.0047" rpy="0 0 0" />
+			<geometry>
+				<mesh filename= "package://coro_descriptions/meshes/table_top.stl"/>
+			</geometry>
+		    <material name="table_top_material">
+				<color rgba="0.615686 0.811765 0.929412 1.0"/>
+			</material>
+		</collision>
+		<visual>
+			<geometry>
+				<mesh filename= "package://coro_descriptions/meshes/table_top.stl"/>
+			</geometry>
+		    <material name="table_top_material">
+				<color rgba="0.615686 0.811765 0.929412 1.0"/>
+			</material>>
+		</visual>
+	</link>
+	<joint name='table_top_to_table_base' type='fixed'>
+		<origin xyz="0.004217 -0.201201 0.97025" rpy="0 0 1.57"/>
+		<parent link="table_base"/>
+		<child link="table_top"/>
 	</joint>
 	<!-- ROBOT -->
@@ -39,19 +69,19 @@
     <link name="cubic_object_link">
 		<visual>
-		<origin xyz="0 0 0" rpy="0 -0 1.5708" />
+		<origin xyz="0 0 0" rpy="0 -0 0" />
 		<geometry>
 		<mesh filename="package://coro_descriptions/meshes/cubic_object.stl"/>
 		</geometry>
 		<material name="link_testing_cube_material">
-		<color rgba="0.615686 0.811765 0.929412 1.0"/>
+			<color rgba="0.615686 0.811765 0.929412 1.0"/>
 		</material>
 		</visual>
 		<collision>
-		<origin xyz="0 0 0" rpy="0 -0 1.5708" />
+		<origin xyz="0 0 0" rpy="0 -0 0" />
 		<geometry>
 		<mesh filename="package://coro_descriptions/meshes/cubic_object.stl"/>
 		</geometry>
 		<material name="link_testing_cube_material">
-		<color rgba="0.615686 0.811765 0.929412 1.0"/>
+			<color rgba="0.615686 0.811765 0.929412 1.0"/>
 		</material>
 		</collision>
@@ -63,5 +93,5 @@
     </link>
 	<joint name='object_to_table' type='fixed'>
-		<origin xyz="0.004217 -0.201201 0.951750" rpy="0 0 0"/>
+		<origin xyz="-0.0049 -0.2062 1.23145" rpy="0 0 0.0206751"/> <!-- Modified elevation along the Z axis to avoid object's interferance with the table top which causes undesired vibrations in gazebo -->
     	<parent link="table_base"/>
     	<child link="cubic_object_link"/>
